File: InputPower.kicad_sch (KiCad schematic)
At the start: 7 parts, among them J1 Wurth 691210910002, J7 Wurth 691210910002, U2 TSR1-2450E, U3 TSR1-2433E

Commit message: Redefined nets - were not setup properly
Parts:
- added C22: 100nF, Capacitor_SMD:C_0805_2012Metric_Pad1.18x1.45mm_HandSolder, symbol Device:C
Connections:
- net GND: now also C7.1, C22.1; no longer C7.2
- net at J1.1, J1.2, U2.1 (Vin)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: now also C7.2, C22.2; no longer C7.1
Other:
- moved on the sheet: C7, C8

Commit message: lots of PCB changes
Parts:
- removed J1, J7: Wurth 691210910002, Robocone Footprints:691210910002, symbol dk_Rectangular-Connectors-Headers-Male-Pins:22-23-2021
- added J1, J2: 691210910002, 691210910002:691210910002, symbol 691210910002:691210910002
Connections:
- net GND: now also J2.2
- net V SUPPLY IN BOTH: now reaches C22.2, C7.2, U2.1 (Vin), U3.1 (Vin)
- net V SUPPLY IN BOTH: now also J1.1, J1.2
- no-connect marks 0 -> 1
